Commit message: plot results

File: assets/urdf/ycb/013_apple.urdf (robot description, URDF)
Before this commit: robot 013_apple, 1 links, 0 joints
Links:
- link _name: geometry collision mesh filename=013_apple/google_16k/textured_vhacd.obj scale=0.9 0.9 0.9; visual mesh filename=013_apple/google_16k/textured.obj scale=0.9 0.9 0.9
